File: dspic30_simple.kicad_pcb (KiCad board)
At the start: 2 copper layers, 95.5 x 65 mm, 22 parts, among them J1 Jack-DC, J2 Conn_01x19_Pin, J4 Conn_01x21_Pin, J6 Conn_PIC_ICSP_ICD, SW1 SW_Push, U1 PIC18F4550-IP, U2 L7805, Y1 Crystal

Commit message: fix GDN not connnected
Parts:
- removed J6: Conn_PIC_ICSP_ICD, Connector_PinSocket_2.54mm:PinSocket_1x06_P2.54mm_Vertical
- added ICSP1: Conn_PIC_ICSP_ICD, Connector_PinSocket_2.54mm:PinSocket_1x06_P2.54mm_Vertical, F.Cu at (171.0, 72.3)
Connections:
- U1 pad 12: unconnected-(U1-VSS-Pad12) -> GND
- U1 pad 31: unconnected-(U1-VSS-Pad31) -> GND
