File: dspic30_simple.kicad_sch (KiCad schematic)
At the start: 21 parts, among them J1 Jack-DC, J2 Conn_01x19_Pin, J4 Conn_01x21_Pin, SW1 SW_Push, U1 PIC18F4550-IP, U2 L7805, Y1 Crystal

Commit message: changes smd component for tht components
Parts:
- removed C3, C4: 18pF, Capacitor_THT:C_Disc_D3.8mm_W2.6mm_P2.50mm, symbol Device:C
- removed Y1: Crystal, Crystal:Crystal_SMD_HC49-SD_HandSoldering, symbol Device:Crystal
- C1, C2: footprint Capacitor_SMD:CP_Elec_8x10 -> Capacitor_THT:CP_Radial_D8.0mm_P3.80mm
- SW1: footprint Button_Switch_SMD:SW_SPST_PTS647_Sx38 -> Button_Switch_THT:SW_PUSH_6mm
- renumbered ICSP to ICSP1
Connections:
- net GND: now also U1.12 (VSS), U1.31 (VSS)
- net RB6: now also U1.14 (RA6/OSC2/CLKO)
- no-connect marks 3 -> 4

Commit message: GND DRC warnings
Connections:
- net GND: no longer J2.14 (Pin_14), J2.15 (Pin_15)
- net RB6: no longer U1.14 (RA6/OSC2/CLKO)
- net RC13: now also J2.15 (Pin_15); no longer J2.13 (Pin_13)
- net CLKI: now reaches U1.13 (OSC1/CLKI)
- net CLKI: now also J2.13 (Pin_13)
- new net RC15: J2.14 (Pin_14), U1.14 (RA6/OSC2/CLKO)
- no-connect marks 4 -> 3
Changed lines of the file:
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@@
 	)
 	(junction
-		(at 234.95 134.62)
-		(diameter 0)
-		(color 0 0 0 0)
-	)
-	(junction
 		(at 245.11 49.53)
 		(diameter 0)
@@
 		(at 107.95 114.3)
 	)
-	(no_connect
-		(at 143.51 63.5)
-	)
-	(wire
-		(pts
-			(xy 234.95 134.62) (xy 234.95 137.16)
-		)
-		(stroke
-			(width 0)
-			(type default)
-		)
-	)
 	(wire
 		(pts
@@
 	(wire
 		(pts
+			(xy 139.7 63.5) (xy 143.51 63.5)
+		)
+		(stroke
+			(width 0)
+			(type default)
+		)
+	)
+	(wire
+		(pts
 			(xy 234.95 114.3) (xy 238.76 114.3)
 		)
@@
 	(wire
 		(pts
+			(xy 237.49 137.16) (xy 234.95 137.16)
+		)
+		(stroke
+			(width 0)
+			(type default)
+		)
+	)
+	(wire
+		(pts
 			(xy 234.95 104.14) (xy 241.3 104.14)
 		)
@@
 	(wire
 		(pts
-			(xy 237.49 132.08) (xy 234.95 132.08)
-		)
-		(stroke
-			(width 0)
-			(type default)
-		)
-	)
-	(wire
-		(pts
 			(xy 203.2 86.36) (xy 199.39 86.36)
 		)
@@
 	(wire
 		(pts
-			(xy 139.7 58.42) (xy 143.51 58.42)
+			(xy 135.89 58.42) (xy 143.51 58.42)
 		)
 		(stroke
@@
 	(wire
 		(pts
+			(xy 234.95 132.08) (xy 242.57 132.08)
+		)
+		(stroke
+			(width 0)
+			(type default)
+		)
+	)
+	(wire
+		(pts
 			(xy 194.31 129.54) (xy 194.31 137.16)
 		)
@@
 	(wire
 		(pts
-			(xy 234.95 134.62) (xy 241.3 134.62)
-		)
-		(stroke
-			(width 0)
-			(type default)
-		)
-	)
-	(wire
-		(pts
 			(xy 234.95 109.22) (xy 238.76 109.22)
 		)
@@
 	(wire
 		(pts
+			(xy 237.49 134.62) (xy 234.95 134.62)
+		)
+		(stroke
+			(width 0)
+			(type default)
+		)
+	)
+	(wire
+		(pts
 			(xy 234.95 116.84) (xy 238.76 116.84)
 		)
@@
 		)
 	)
+	(label "RC15"
+		(at 237.49 134.62 0)
+		(fields_autoplaced yes)
+		(effects
+			(font
+				(size 1.27 1.27)
+			)
+			(justify left bottom)
+		)
+	)
 	(label "AVSS"
 		(at 137.16 83.82 0)
@@
 		)
 	)
-	(label "RB6"
-		(at 139.7 58.42 0)
+	(label "RC15"
+		(at 135.89 58.42 0)
 		(fields_autoplaced yes)
 		(effects
@@
 		)
 	)
+	(label "CLKI"
+		(at 242.57 132.08 0)
+		(fields_autoplaced yes)
+		(effects
+			(font
+				(size 1.27 1.27)
+			)
+			(justify left bottom)
+		)
+	)
 	(label "RB4"
 		(at 139.7 53.34 0)
@@
 		)
 	)
-	(label "RC13"
-		(at 237.49 132.08 0)
-		(fields_autoplaced yes)
-		(effects
-			(font
-				(size 1.27 1.27)
-			)
-			(justify left bottom)
-		)
-	)
 	(label "PGD"
 		(at 208.28 55.88 0)
@@
 		)
 	)
+	(label "RC13"
+		(at 237.49 137.16 0)
+		(fields_autoplaced yes)
+		(effects
+			(font
+				(size 1.27 1.27)
+			)
+			(justify left bottom)
+		)
+	)
 	(label "VD2"
 		(at 171.45 33.02 0)
@@
 		)
 	)
+	(label "CLKI"
+		(at 139.7 63.5 0)
+		(fields_autoplaced yes)
+		(effects
+			(font
+				(size 1.27 1.27)
+			)
+			(justify left bottom)
+		)
+	)
 	(label "VD3"
 		(at 194.31 133.35 0)
@@
 					(unit 1)
 				)
-			)
-		)
-	)
-	(symbol
-		(lib_id "power:GND")
-		(at 241.3 134.62 0)
-		(unit 1)
-		(exclude_from_sim no)
-		(in_bom yes)
-		(on_board yes)
-		(dnp no)
-		(property "Reference" "#PWR011"
-			(at 241.3 140.97 0)
-			(effects
-				(font
-					(size 1.27 1.27)
-				)
-				(hide yes)
-			)
-		)
-		(property "Value" "GND"
-			(at 241.3 139.7 0)
-			(effects
-				(font
-					(size 1.27 1.27)
-				)
-			)
-		)
-		(property "Footprint" ""
-			(at 241.3 134.62 0)
-			(effects
-				(font
-					(size 1.27 1.27)
-				)
-				(hide yes)
-			)
-		)
-		(property "Datasheet" ""
-			(at 241.3 134.62 0)
-			(effects
-				(font
-					(size 1.27 1.27)
-				)
-				(hide yes)
-			)
-		)
-		(property "Description" "Power symbol creates a global label with name \"GND\" , ground"
-			(at 241.3 134.62 0)
-			(effects
-				(font
-					(size 1.27 1.27)
-				)
-				(hide yes)
-			)
-		)
-		(pin "1"
-		)
-		(instances
-			(project ""
-				(path "/c57c8b8a-cb5c-45d3-8c1c-ff7cf62f6723"
-					(reference "#PWR011")
-					(unit 1)
-				)
